File: ESPBreakotBoard-Min-Cutout.kicad_sch (KiCad schematic)
At the start: 13 parts, among them J1 Screw_Terminal_01x02, J2 Conn_01x09_Male, J3 Conn_01x09_Male, U1 AMS1117-3.3, U2 ESP-07

Commit message: v4r2: Fixed Silkscreen and 3D Models
Parts:
- added H1: M2, MountingHole:MountingHole_2.2mm_M2_Pad_Via, symbol Mechanical:MountingHole
Changed lines of the file:
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@@
     (pin "2")
+  )
+  (symbol (lib_id "Mechanical:MountingHole") (at 95.885 76.2 0) (unit 1)
+    (in_bom yes) (on_board yes) (fields_autoplaced)
+    (property "Reference" "H1" (id 0) (at 99.06 74.9299 0)
+      (effects (font (size 1.27 1.27)) (justify left))
+    )
+    (property "Value" "M2" (id 1) (at 99.06 77.4699 0)
+      (effects (font (size 1.27 1.27)) (justify left))
+    )
+    (property "Footprint" "MountingHole:MountingHole_2.2mm_M2_Pad_Via" (id 2) (at 95.885 76.2 0)
+      (effects (font (size 1.27 1.27)) hide)
+    )
+    (property "Datasheet" "~" (id 3) (at 95.885 76.2 0)
+      (effects (font (size 1.27 1.27)) hide)
+    )
   )
   (sheet_instances
@@
       (reference "C3") (unit 1) (value "100nF") (footprint "Capacitor_SMD:C_0805_2012Metric_Pad1.18x1.45mm_HandSolder")
     )
+    (path "/4a333138-062a-4541-87e1-d6ef03b1e3dd"
+      (reference "H1") (unit 1) (value "M2") (footprint "MountingHole:MountingHole_2.2mm_M2_Pad_Via")
+    )
     (path "/00000000-0000-0000-0000-000060dae008"
